File: hardware/MSXIoT/MSXIoT_bus.brd (EAGLE design)
At the start: 102.5 x 81.3 mm, 17 parts, among them IC1 74LS00N, IC2 74LS138N, IC3 74LS138N, IC4 74LS245N

Commit message: marzo2021
Parts:
- removed E$1: (no value), ESP32-WROOM-32:MODULE_ESP32-WROOM-32
- added C7: (no value), resistor:153CLV-0505
- added JP6, JP7: PINHD-1X6, Connector:1X06
- added JP8: PINHD-1X5/90, Connector:1X05/90
- added JP9: PINHD-2X3, Connector:2X03
- added Q1, Q2: NPN__SOT-23, Transistor:SOT95P237X112-3N
- added R1, R2: (no value), resistor:0204/5
- added U1: ESP32-WROOM-32, ESP32-WROOM-32:MODULE_ESP32-WROOM-32
- C1: value (none) -> 100nf
- C2, C3, C4, C5: value (none) -> 100n
- C6: value (none) -> 100uF
- moved C3 8.89 mm to (68.6, 66.7)
- moved IC1 8.89 mm to (68.6, 55.9)
- moved C2 5.08 mm to (80.1, 66.7)
- moved IC3 5.08 mm to (80.0, 54.6)
- moved IC4 2.84 mm to (43.2, 49.5)
- moved C4 1.27 mm to (43.2, 66.7)
- moved JP2 1.27 mm to (34.3, 41.9)
- moved JP3 1.27 mm to (34.3, 58.4)
- moved JP4 1.27 mm to (24.1, 41.9)
- moved JP5 1.27 mm to (24.1, 58.4)
- moved C1 1.27 mm to (91.6, 66.7)
- moved IC2 1.27 mm to (91.4, 54.6)
Connections:
- removed net A15: IC5.3
- removed net A16: IC5.2
- new net 3V3: JP4.3, JP5.3, JP7.3, U1.2
- new net A03V3: JP7.1, U1.24
- new net D_IO0: JP5.6, U1.37
- new net D_IO1: JP5.5, U1.36
- new net D_IO2: JP5.2, U1.33
- new net D_IO3: JP5.1, U1.31
- new net D_IO4: JP4.6, U1.30
- new net D_IO5: JP4.5, U1.28
- new net D_IO6: JP4.2, U1.27
- new net D_IO7: JP4.1, U1.26
- new net EN: IC1.9, JP6.2
- new net EN3V3: JP7.5, U1.16
- new net INT3V3: C7.+, JP7.2, U1.7
- new net N$14: JP8.5, U1.34
- new net N$15: U1.25
- new net N$16: JP8.1, Q2.1, R1.1
- new net N$17: Q1.2, R1.2
- new net RD3V3: JP7.6, U1.6
- new net SA15: IC5.3, JP9.3
- new net SA16: IC5.2, JP9.4
- net A0: now also JP6.6
- net GND: now also IC5.30, JP6.3, JP7.4, JP8.3, JP9.1, JP9.2, U1.1, U1.15, U1.38, U1.39_1, U1.39_10, U1.39_11, U1.39_12, U1.39_13, U1.39_14, U1.39_15, U1.39_16, U1.39_17, U1.39_18, U1.39_19, U1.39_2, U1.39_20, U1.39_21, U1.39_3, U1.39_4, U1.39_5, U1.39_6, U1.39_7, U1.39_8, U1.39_9
- net INT: now also JP6.5
- net N$13: now also JP8.4, U1.35; no longer IC1.9
- net N$18: now also Q2.2, R2.2; no longer JP4.3
- net N$19: now also JP8.2, Q1.1, R2.1; no longer JP5.3
- net RD: now also JP6.1
- net VCC: now also IC5.31, JP6.4, JP9.5, JP9.6
Routing:
- net GND: track 261.3 -> 397.0 mm, vias 3 -> 8
- net 3V3: track 0.00 -> 94.7 mm, vias 0 -> 3
- net RD3V3: track 0.00 -> 74.0 mm, vias 0 -> 1
- net EN3V3: track 0.00 -> 61.7 mm, vias 0 -> 1
- net INT3V3: track 0.00 -> 58.1 mm, vias 0 -> 1
- net VCC: track 219.8 -> 264.4 mm, vias 0 -> 7
- net A03V3: track 0.00 -> 44.4 mm, vias 0 -> 1
- net A0: track 79.2 -> 117.7 mm
- net SA16: track 0.00 -> 29.2 mm, vias 0 -> 2
- net RD: track 76.1 -> 104.5 mm
- net SA15: track 0.00 -> 20.7 mm
- net N$14: track 0.00 -> 19.0 mm, vias 0 -> 1
- net N$13: track 0.00 -> 18.7 mm, vias 0 -> 1
- net D_IO0: track 0.00 -> 17.2 mm
- net D_IO1: track 0.00 -> 16.1 mm
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Other:
- board text added: "MSX-IoT"
- board text added: "v1.1 2020"
