File: hardware/MSXIoT/MSXIoT_bus.sch (EAGLE design)
At the start: 17 parts, among them IC1 74LS00N, IC2 74LS138N, IC3 74LS138N, IC4 74LS245N, U1 ESP32-WROOM-32

Commit message: marzo2021
Parts:
- added C7: (no value), resistor:CPOL-US153CLV-0505
- added JP6, JP7: PINHD-1X6, Connector:PINHD-1X6
- added JP8: PINHD-1X5/90, Connector:PINHD-1X5/90
- added JP9: PINHD-2X3, Connector:PINHD-2X3
- added Q1, Q2: NPN__SOT-23, Transistor:NPN__SOT-23
- added R1, R2: (no value), resistor:R-US_0204/5
- C1: value (none) -> 100nf
- C2, C3, C4, C5: value (none) -> 100n
- C6: value (none) -> 100uF
Connections:
- removed net A15: IC5.A15
- removed net A16: IC5.A16
- new net 3V3: JP4.3, JP5.3, JP7.3
- new net A03V3: JP7.1, U1.IO2
- new net D_IO0: JP5.6, U1.IO23
- new net D_IO1: JP5.5, U1.IO22
- new net D_IO2: JP5.2, U1.IO21
- new net D_IO3: JP5.1, U1.IO19
- new net D_IO4: JP4.6, U1.IO18
- new net D_IO5: JP4.5, U1.IO17
- new net D_IO6: JP4.2, U1.IO16
- new net D_IO7: JP4.1, U1.IO4
- new net EN: IC1C.I0, JP6.2
- new net EN3V3: JP7.5, U1.IO13
- new net INT3V3: C7.+, JP7.2, U1.IO35
- new net N$14: JP8.5, U1.RXD0
- new net N$15: U1.IO0
- new net N$16: JP8.1, Q2.E, R1.1
- new net N$17: Q1.B, R1.2
- new net RD3V3: JP7.6, U1.IO34
- new net SA15: IC5.A15, JP9.3
- new net SA16: IC5.A16, JP9.4
- net A0: now also JP6.6
- net GND: now also IC5.GND, IC5.NC, JP6.3, JP7.4, JP8.3, JP9.1, JP9.2
- net INT: now also JP6.5
- net N$13: now also JP8.4, U1.TXD0; no longer IC1C.I0
- net N$18: now also Q2.B, R2.2; no longer JP4.3
- net N$19: now also JP8.2, Q1.E, R2.1; no longer JP5.3
- net RD: now also JP6.1
- net VCC: now also IC5.!PGM, IC5.VCC, JP6.4, JP9.5, JP9.6
Other:
- moved on the sheet: U1
